Commit message: edit some urdf robot

File: mobile_robot_autonomous_navigation/urdf/mobile_robot_v2.xacro (robot description, xacro)
@@ -1,7 +1,7 @@
 <?xml version="1.0"?>
 <robot xmlns:xacro="http://www.ros.org/wiki/xacro" name="mobile_robot">
-  <xacro:property name="base_width" value="0.3"/>
-  <xacro:property name="base_len" value="0.4"/>
-  <xacro:property name="base_height" value="0.12"/>
+  <xacro:property name="base_width" value="0.4"/>
+  <xacro:property name="base_len" value="0.6"/>
+  <xacro:property name="base_height" value="0.2"/>
   <xacro:property name="wheel_radius" value="0.085"/>
   <xacro:property name="base_wheel_gap" value="0.02"/>
@@ -49,5 +49,5 @@
      <parent link="dummy"/>
      <child link="base_footprint"/>
-     </joint>
+  </joint>
   <link name="base_link">
     <xacro:box_inertia m="1" w="${base_len}" h="${base_width}" d="0.01"/>
@@ -138,5 +138,5 @@
     <parent link="base_link" />
     <child link="lidar" />
-    <origin xyz="0.0 0.0 0.12" rpy="0 0 3.14159" />
+    <origin xyz="0.0 0.0 0.40" rpy="0 0 3.14159" />
   </joint>
   <link name="lidar">
