Commit message: rename to autonomous_mobile_robot_navigation

File: autonomous_mobile_robot_navigation/urdf/mobile_robot.xacro (robot description, xacro)
@@ -40,5 +40,5 @@
       <origin rpy="0 0 0" xyz="0.03 0 -0.026"/>
       <geometry>
-        <mesh filename="package://mobile_robot_autonomous_navigation/stl/Chasis.stl" scale="0.001 0.001 0.001"/>
+        <mesh filename="package://autonomous_mobile_robot_navigation/stl/Chasis.stl" scale="0.001 0.001 0.001"/>
       </geometry>
       <material name="white"/>
@@ -47,5 +47,5 @@
       <origin rpy="0 0 0" xyz="0.03 0 -0.026"  />
       <geometry>
-        <mesh filename="package://mobile_robot_autonomous_navigation/stl/Chasis.stl" scale="0.001 0.001 0.001" />
+        <mesh filename="package://autonomous_mobile_robot_navigation/stl/Chasis.stl" scale="0.001 0.001 0.001" />
       </geometry>
     </collision>
@@ -61,5 +61,5 @@
       <origin rpy="0 0 0" xyz="0.11 0.059 -0.04"/>
       <geometry>
-        <mesh filename="package://mobile_robot_autonomous_navigation/stl/Wheel.stl" scale="0.001 0.001 0.001"/>
+        <mesh filename="package://autonomous_mobile_robot_navigation/stl/Wheel.stl" scale="0.001 0.001 0.001"/>
       </geometry>
       <material name="black"/>
@@ -68,5 +68,5 @@
       <origin rpy="0 0 0" xyz="0.11 0.059 -0.04"/>
       <geometry>
-        <mesh filename="package://mobile_robot_autonomous_navigation/stl/Wheel.stl" scale="0.001 0.001 0.001" />
+        <mesh filename="package://autonomous_mobile_robot_navigation/stl/Wheel.stl" scale="0.001 0.001 0.001" />
       </geometry>
     </collision>
@@ -82,5 +82,5 @@
       <origin rpy="0 0 0" xyz="0.133 0.059 -0.04"/>
       <geometry>
-        <mesh filename="package://mobile_robot_autonomous_navigation/stl/Wheel.stl" scale="0.001 0.001 0.001"/>
+        <mesh filename="package://autonomous_mobile_robot_navigation/stl/Wheel.stl" scale="0.001 0.001 0.001"/>
       </geometry>
       <material name="black"/>
@@ -89,5 +89,5 @@
       <origin rpy="0 0 0" xyz="0.133 0.059 -0.04"/>
       <geometry>
-        <mesh filename="package://mobile_robot_autonomous_navigation/stl/Wheel.stl" scale="0.001 0.001 0.001" />
+        <mesh filename="package://autonomous_mobile_robot_navigation/stl/Wheel.stl" scale="0.001 0.001 0.001" />
       </geometry>
     </collision>
@@ -102,5 +102,5 @@
       <origin rpy="0 0 -1.5708" xyz="0.084 -0.242 -0.098"/>
       <geometry>
-        <mesh filename="package://mobile_robot_autonomous_navigation/stl/RpLidar.stl" scale="0.001 0.001 0.001"/>
+        <mesh filename="package://autonomous_mobile_robot_navigation/stl/RpLidar.stl" scale="0.001 0.001 0.001"/>
       </geometry>
       <material name="blue"/>
@@ -109,5 +109,5 @@
       <origin rpy="0 0 0" xyz="0.242 0.084 -0.098"  />
       <geometry>
-        <mesh filename="package://mobile_robot_autonomous_navigation/stl/RpLidar.stl" scale="0.001 0.001 0.001" />
+        <mesh filename="package://autonomous_mobile_robot_navigation/stl/RpLidar.stl" scale="0.001 0.001 0.001" />
       </geometry>
     </collision>

File: autonomous_mobile_robot_navigation/urdf/mobile_robot_v2.xacro (robot description, xacro)
@@ -10,5 +10,5 @@
   <xacro:property name="caster_wheel_radius" value="0.0375"/>
   <xacro:property name="caster_wheel_joint_offset" value="0.12"/>
-  <xacro:include filename="$(find mobile_robot_autonomous_navigation)/urdf/mobile_robot_v2_gazebo_plugins.xacro"/>
+  <xacro:include filename="$(find autonomous_mobile_robot_navigation)/urdf/mobile_robot_v2_gazebo_plugins.xacro"/>
   <material name="blue">
     <color rgba="0 0 0.8 1"/>
